File: BaseTag.sch (EAGLE design)
At the start: 27 parts, among them U1 BQ25504, U3 MSP430FR2512IPW16RSOIC

Commit message: alpha layout
Parts:
- added C10, C11, C12, C13, C14, C15, C16, C17, C9: 11mF, Nelson-RLCD:C
- added D3, D4: 44mA@0.5V, Nelson-IC:SOLAR-CELL
- added SV3: (no value), con-lstb:MA04-1
- C1: device Nelson-RLCD:C11MF1210 -> Nelson-RLCD:C
- R1: value 4.42MOhm -> 4.42MOhom
Connections:
- removed net N$8: C1.+, U1.VBAT
- new net VBAT: C1.+, C10.+, C11.+, C12.+, C13.+, C14.+, C15.+, C16.+, C17.+, C9.+, SV3.4, U1.VBAT
- new net VIN: C2.+, D1.+, D3.+, L1.P$1, R1.P$2, SV3.2, U1.VIN_DC
- net +3V3: now also C3.+; no longer C3.-
- net GND: now also C10.-, C11.-, C12.-, C13.-, C14.-, C15.-, C16.-, C17.-, C3.-, C9.-, D4.-, SV3.1, SV3.3; no longer C3.+
- net N$1: now also D3.-, D4.+; no longer C2.+, D1.+, L1.P$1, R1.P$2, U1.VIN_DC
Other:
- moved on the sheet: C3

Commit message: prep for 1" branch
Parts:
- added C18, C19, C20, C21, C22, C23, C24, C25, C26, C27, C28, C29, C30, C31: 11mF, Nelson-RLCD:C
- added R11, R12: R, Nelson-RLCD:R
Connections:
- new net N$8: R12.P$1, U1.VBAT
- new net VIN_: C2.+, L1.P$1, R1.P$2, R11.P$2, U1.VIN_DC
- net GND: now also C18.-, C19.-, C20.-, C21.-, C22.-, C23.-, C24.-, C25.-, C26.-, C27.-, C28.-, C29.-, C30.-, C31.-
- net VBAT: now also C18.+, C19.+, C20.+, C21.+, C22.+, C23.+, C24.+, C25.+, C26.+, C27.+, C28.+, C29.+, C30.+, C31.+, R12.P$2; no longer U1.VBAT
- net VIN: now also R11.P$1; no longer C2.+, L1.P$1, R1.P$2, U1.VIN_DC
Other:
- moved on the sheet: D1, D2, D3, D4

Commit message: prelim oneinch
Parts:
- removed C30, C31: 11mF, Nelson-RLCD:C
- removed D3, D4: 44mA@0.5V, Nelson-IC:SOLAR-CELL
- removed SV1, SV3: (no value), con-lstb:MA04-1
- removed SV2: (no value), con-lstb:MA10-1
- removed TP1, TP2: TPB1,27, testpad:TPB1,27
- added J1: PIN-1-10, Nelson-con:PIN-1-10
- added J2, J3: PIN-1-4, Nelson-con:PIN-1-4
- added J4: PIN-1-2, Nelson-con:PIN-1-2
Connections:
- removed net N$1: D3.-, D4.+
- removed net N$12: SV2.10, U3.2.2/TA1.1/SYNC/A4
- removed net N$13: SV2.9, U3.P1.7/UCA0STE/TDO/CAP0.3
- removed net N$14: SV2.8, U3.P1.6/UCA0CLK/TA0CLK/TDI/TCLK/CAP0.2
- removed net N$15: SV2.7, U3.P1.5/UCA0RXD/UCA0SOMI/TA0.2/TMS/CAP0.1
- removed net N$16: SV2.6, U3.P1.4/UCA0TXD/UCA0SIMO/TA0.1/TCK/CAP0.0
- removed net N$17: SV2.5, U3.P1.3/UCB0SOMI/UCB0SCL/MCLK/A3/CAP1.3
- removed net N$18: SV2.4, U3.P1.2/UCB0SIMO/UCB0SDA/SMCLK/A2/VEREF-/CAP1.2
- removed net N$19: SV2.3, U3.P1.1/UCB0CLK/ACLK/A1/VREF+/CAP1.1
- new net 1.1: J1.P$3, U3.P1.1/UCB0CLK/ACLK/A1/VREF+/CAP1.1
- new net 1.2: J1.P$4, U3.P1.2/UCB0SIMO/UCB0SDA/SMCLK/A2/VEREF-/CAP1.2
- new net 1.3: J1.P$5, U3.P1.3/UCB0SOMI/UCB0SCL/MCLK/A3/CAP1.3
- new net 1.4: J1.P$6, U3.P1.4/UCA0TXD/UCA0SIMO/TA0.1/TCK/CAP0.0
- new net 1.5: J1.P$7, U3.P1.5/UCA0RXD/UCA0SOMI/TA0.2/TMS/CAP0.1
- new net 1.6: J1.P$8, U3.P1.6/UCA0CLK/TA0CLK/TDI/TCLK/CAP0.2
- new net 1.7: J1.P$9, U3.P1.7/UCA0STE/TDO/CAP0.3
- new net 2.2: J1.P$10, U3.2.2/TA1.1/SYNC/A4
- net +3V3: now also J1.P$1, J2.P$2; no longer SV1.2, SV2.1
- net GND: now also J1.P$2, J2.P$1, J3.P$1, J3.P$3; no longer C30.-, C31.-, D4.-, SV1.1, SV2.2, SV3.1, SV3.3
- net RESET: now also J4.P$2; no longer TP1.TP
- net RX: now also J2.P$4; no longer SV1.4
- net TEST: now also J4.P$1; no longer TP2.TP
- net TX: now also J2.P$3; no longer SV1.3
- net VBAT: now also J3.P$4; no longer C30.+, C31.+, SV3.4
- net VIN: now also J3.P$2; no longer D3.+, SV3.2
Other:
- moved on the sheet: C18, C19, C20, C21, C22, C23, C24, C25, C26, C27, C28, C29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
