File: BaseTag.brd (EAGLE design)
At the start: 100 x 80 mm, 27 parts, among them U1 BQ25504, U3 MSP430FR2512IPW16RSOIC

Commit message: alpha layout
Parts:
- added C10, C11, C12, C13, C14, C15, C16, C17, C9: 11mF, Nelson-RLCD:CPH3225A-2K
- added D3, D4: 44mA@0.5V, Nelson-IC:KXOB22-12X1F
- added SV3: (no value), con-lstb:MA04-1
- C1: device Nelson-RLCD:CAPCP6425X90 -> Nelson-RLCD:CPH3225A-2K
- R1: value 4.42MOhm -> 4.42MOhom
- moved SV2 327.6 mm to (17.8, 33.0)
- moved D2 304.6 mm to (14.0, 17.8), flipped to the bottom, turned to 90 degrees
- moved SV1 284.7 mm to (22.9, 2.54)
- moved C8 280.6 mm to (29.5, 24.6), turned to 135 degrees
- moved TP2 278.9 mm to (28.4, 8.89), turned to 270 degrees
- moved R10 277.0 mm to (30.0, 11.9), turned to 90 degrees
- moved TP1 270.8 mm to (30.2, 8.89), turned to 270 degrees
- moved C7 267.9 mm to (32.1, 13.2)
- moved U3 264.9 mm to (31.5, 18.3), turned to 90 degrees
- moved C6 264.2 mm to (32.1, 11.9)
- moved C5 261.8 mm to (7.49, 19.4)
- moved R9 252.4 mm to (10.8, 15.9)
- moved R8 238.3 mm to (10.8, 14.5)
- moved R7 224.3 mm to (10.8, 13.2)
- moved R4 209.0 mm to (8.38, 10.7), turned to 180 degrees
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Connections:
- removed net N$8: C1.+, U1.14
- new net VBAT: C1.+, C10.+, C11.+, C12.+, C13.+, C14.+, C15.+, C16.+, C17.+, C9.+, SV3.4, U1.14
- new net VIN: C2.+, D1.+, D3.+, L1.P$1, R1.-, SV3.2, U1.2
- net +3V3: now also C3.+; no longer C3.-
- net GND: now also C10.-, C11.-, C12.-, C13.-, C14.-, C15.-, C16.-, C17.-, C3.-, C9.-, D4.-, SV3.1, SV3.3; no longer C3.+
- net N$1: now also D3.-, D4.+; no longer C2.+, D1.+, L1.P$1, R1.-, U1.2
Routing:
- net +3V3: track 0.00 -> 90.1 mm
- net VIN: track 0.00 -> 56.6 mm, vias 0 -> 1
- net N$19: track 0.00 -> 30.3 mm
- net VBAT_OK: track 0.00 -> 24.9 mm, vias 0 -> 2
- net VBAT: track 0.00 -> 24.4 mm, vias 0 -> 1
- net TX: track 0.00 -> 22.6 mm
- net N$18: track 0.00 -> 21.8 mm
- net N$17: track 0.00 -> 20.0 mm
- net N$16: track 0.00 -> 20.0 mm
- net N$15: track 0.00 -> 17.9 mm
- net N$14: track 0.00 -> 16.4 mm
- net RX: track 0.00 -> 16.1 mm
- net N$13: track 0.00 -> 14.5 mm
- net N$12: track 0.00 -> 13.7 mm
- net RESET: track 0.00 -> 9.01 mm
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- added copper zone on layer 1, net GND
- added copper zone on layer 16, net GND
- added copper zone on layer 1, net VBAT
Other:
- board size 100 x 80 mm -> 35.6 x 35.6 mm
- board text added: "todo check crystal check super cap layout label pins"

Commit message: prep for 1" branch
Parts:
- added C18, C19, C20, C21, C22, C23, C24, C25, C26, C27, C28, C29, C30, C31: 11mF, Nelson-RLCD:CPH3225A-2K
- added R11, R12: R, Nelson-RLCD:0603
- moved C10 9.18 mm to (20.6, 20.8)
- moved C11 9.18 mm to (23.6, 20.8)
- moved C15 9.18 mm to (26.7, 20.8)
- moved C16 9.18 mm to (14.5, 20.8)
- moved C9 9.18 mm to (17.5, 20.8)
- moved C1 6.14 mm to (17.5, 25.7)
- moved C12 6.14 mm to (20.6, 25.7)
- moved C13 6.14 mm to (23.6, 25.7)
- moved C14 6.14 mm to (26.7, 25.7)
- moved C17 6.14 mm to (14.5, 25.7)
- moved C3 1.85 mm to (8.00, 18.9)
- moved C5 1.85 mm to (8.00, 17.7)
- moved C4 1.85 mm to (4.57, 12.1)
- moved R2 1.85 mm to (3.30, 12.1)
- moved R6 1.85 mm to (6.35, 8.12)
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Connections:
- new net N$8: R12.+, U1.14
- new net VIN_: C2.+, L1.P$1, R1.-, R11.-, U1.2
- net GND: now also C18.-, C19.-, C20.-, C21.-, C22.-, C23.-, C24.-, C25.-, C26.-, C27.-, C28.-, C29.-, C30.-, C31.-
- net VBAT: now also C18.+, C19.+, C20.+, C21.+, C22.+, C23.+, C24.+, C25.+, C26.+, C27.+, C28.+, C29.+, C30.+, C31.+, R12.-; no longer U1.14
- net VIN: now also R11.+; no longer C2.+, L1.P$1, R1.-, U1.2
Routing:
- net VBAT: track 24.4 -> 0.00 mm, vias 1 -> 0
- net VIN_: track 0.00 -> 18.6 mm
- net +3V3: track 90.1 -> 94.5 mm
- net N$8: track 0.00 -> 4.43 mm
- net GND: track 0.00 -> 2.63 mm
- net N$17: track 20.0 -> 22.6 mm
- net N$18: track 21.8 -> 24.4 mm
- net N$15: track 17.9 -> 20.0 mm
- net N$19: track 30.3 -> 32.3 mm
- net N$16: track 20.0 -> 21.8 mm
- net N$14: track 16.4 -> 17.8 mm
- net TEST: track 7.72 -> 8.99 mm
- net N$13: track 14.5 -> 15.7 mm
- net VIN: track 56.6 -> 57.7 mm
- removed copper zone on layer 1, net VBAT

Commit message: prelim oneinch
Parts:
- removed C30, C31: 11mF, Nelson-RLCD:CPH3225A-2K
- removed D3, D4: 44mA@0.5V, Nelson-IC:KXOB22-12X1F
- removed SV1, SV3: (no value), con-lstb:MA04-1
- removed SV2: (no value), con-lstb:MA10-1
- removed TP1, TP2: TPB1,27, testpad:B1,27
- added J1: PIN-1-10, Nelson-con:PIN-100MIL-1-10
- added J2, J3: PIN-1-4, Nelson-con:PIN-100MIL-1-4
- added J4: PIN-1-2, Nelson-con:PIN-100MIL-1-2
- moved C28 25.2 mm to (23.4, 6.10), turned to 270 degrees
- moved C16 19.7 mm to (22.4, 2.79), flipped to the bottom, turned to 180 degrees
- moved C29 19.5 mm to (20.3, 6.10)
- moved C8 19.0 mm to (14.2, 15.4)
- moved C6 18.3 mm to (15.9, 3.56)
- moved C7 18.3 mm to (15.9, 4.83)
- moved R10 18.3 mm to (13.7, 3.56)
- moved U3 18.3 mm to (15.2, 9.91)
- moved C17 14.9 mm to (20.3, 11.9), flipped to the bottom
- moved C14 14.1 mm to (23.4, 11.9), flipped to the bottom
- moved C15 14.1 mm to (23.4, 7.11), flipped to the bottom
- moved C13 10.9 mm to (17.3, 16.8), flipped to the bottom, turned to 270 degrees
- moved C18 10.4 mm to (20.3, 7.11), flipped to the bottom, turned to 270 degrees
- moved C22 10.2 mm to (20.3, 20.6), turned to 90 degrees
- moved C12 8.89 mm to (20.3, 16.8), flipped to the bottom, turned to 270 degrees
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Connections:
- removed net N$1: D3.-, D4.+
- removed net N$12: SV2.10, U3.9
- removed net N$13: SV2.9, U3.10
- removed net N$14: SV2.8, U3.11
- removed net N$15: SV2.7, U3.12
- removed net N$16: SV2.6, U3.13
- removed net N$17: SV2.5, U3.15
- removed net N$18: SV2.4, U3.16
- removed net N$19: SV2.3, U3.1
- new net 1.1: J1.3, U3.1
- new net 1.2: J1.4, U3.16
- new net 1.3: J1.5, U3.15
- new net 1.4: J1.6, U3.13
- new net 1.5: J1.7, U3.12
- new net 1.6: J1.8, U3.11
- new net 1.7: J1.9, U3.10
- new net 2.2: J1.10, U3.9
- net +3V3: now also J1.1, J2.2; no longer SV1.2, SV2.1
- net GND: now also J1.2, J2.1, J3.1, J3.3; no longer C30.-, C31.-, D4.-, SV1.1, SV2.2, SV3.1, SV3.3
- net RESET: now also J4.2; no longer TP1.TP
- net RX: now also J2.4; no longer SV1.4
- net TEST: now also J4.1; no longer TP2.TP
- net TX: now also J2.3; no longer SV1.3
- net VBAT: now also J3.4; no longer C30.+, C31.+, SV3.4
- net VIN: now also J3.2; no longer D3.+, SV3.2
Routing:
- net +3V3: track 94.5 -> 42.4 mm, vias 0 -> 2
- net VBAT: track 0.00 -> 51.7 mm, vias 0 -> 3
- net VIN: track 57.7 -> 6.10 mm, vias 1 -> 0
- net N$19: track 32.3 -> 0.00 mm
- net N$18: track 24.4 -> 0.00 mm
- net N$17: track 22.6 -> 0.00 mm
- net N$16: track 21.8 -> 0.00 mm
- net 1.1: track 0.00 -> 21.6 mm
- net N$15: track 20.0 -> 0.00 mm
- net N$14: track 17.8 -> 0.00 mm
- net 2.2: track 0.00 -> 16.9 mm
- net N$13: track 15.7 -> 0.00 mm
- net 1.7: track 0.00 -> 15.2 mm
- net VBAT_OK: track 25.1 -> 10.1 mm
- net 1.2: track 0.00 -> 14.2 mm
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- added copper zone on layer 1, net VBAT
- added copper zone on layer 16, net VBAT
Other:
- board size 35.6 x 35.6 mm -> 25.4 x 25.4 mm
- board text added: "1.1"
- board text added: "1.2"
- board text added: "1.3"
- board text added: "1.4"
- board text added: "1.5"
- board text added: "1.6"
- board text added: "1.7"
- board text added: "2.2"
- board text added: "3v"
- board text added: "bat"
- board text added: "gnd"
- board text added: "in"
- board text added: "rst"
- board text added: "rx"
- board text added: "test"
- board text added: "tx"
- board text removed: "todo check crystal check super cap layout label pins"

Commit message: v1 order
Routing:
- net VBAT: track 51.7 -> 52.4 mm
Changed lines of the file:
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@@
 <layer number="25" name="tNames" color="7" fill="1" visible="yes" active="yes"/>
 <layer number="26" name="bNames" color="7" fill="1" visible="yes" active="yes"/>
-<layer number="27" name="tValues" color="7" fill="1" visible="yes" active="yes"/>
-<layer number="28" name="bValues" color="7" fill="1" visible="yes" active="yes"/>
-<layer number="29" name="tStop" color="7" fill="3" visible="yes" active="yes"/>
-<layer number="30" name="bStop" color="7" fill="6" visible="yes" active="yes"/>
-<layer number="31" name="tCream" color="7" fill="4" visible="yes" active="yes"/>
-<layer number="32" name="bCream" color="7" fill="5" visible="yes" active="yes"/>
-<layer number="33" name="tFinish" color="6" fill="3" visible="yes" active="yes"/>
-<layer number="34" name="bFinish" color="6" fill="6" visible="yes" active="yes"/>
-<layer number="35" name="tGlue" color="7" fill="4" visible="yes" active="yes"/>
-<layer number="36" name="bGlue" color="7" fill="5" visible="yes" active="yes"/>
-<layer number="37" name="tTest" color="7" fill="1" visible="yes" active="yes"/>
-<layer number="38" name="bTest" color="7" fill="1" visible="yes" active="yes"/>
+<layer number="27" name="tValues" color="7" fill="1" visible="no" active="yes"/>
+<layer number="28" name="bValues" color="7" fill="1" visible="no" active="yes"/>
+<layer number="29" name="tStop" color="7" fill="3" visible="no" active="yes"/>
+<layer number="30" name="bStop" color="7" fill="6" visible="no" active="yes"/>
+<layer number="31" name="tCream" color="7" fill="4" visible="no" active="yes"/>
+<layer number="32" name="bCream" color="7" fill="5" visible="no" active="yes"/>
+<layer number="33" name="tFinish" color="6" fill="3" visible="no" active="yes"/>
+<layer number="34" name="bFinish" color="6" fill="6" visible="no" active="yes"/>
+<layer number="35" name="tGlue" color="7" fill="4" visible="no" active="yes"/>
+<layer number="36" name="bGlue" color="7" fill="5" visible="no" active="yes"/>
+<layer number="37" name="tTest" color="7" fill="1" visible="no" active="yes"/>
+<layer number="38" name="bTest" color="7" fill="1" visible="no" active="yes"/>
 <layer number="39" name="tKeepout" color="4" fill="11" visible="yes" active="yes"/>
 <layer number="40" name="bKeepout" color="1" fill="11" visible="yes" active="yes"/>
 <layer number="41" name="tRestrict" color="4" fill="10" visible="yes" active="yes"/>
 <layer number="42" name="bRestrict" color="1" fill="10" visible="yes" active="yes"/>
-<layer number="43" name="vRestrict" color="2" fill="10" visible="yes" active="yes"/>
-<layer number="44" name="Drills" color="7" fill="1" visible="yes" active="yes"/>
-<layer number="45" name="Holes" color="7" fill="1" visible="yes" active="yes"/>
-<layer number="46" name="Milling" color="3" fill="1" visible="yes" active="yes"/>
-<layer number="47" name="Measures" color="7" fill="1" visible="yes" active="yes"/>
-<layer number="48" name="Document" color="7" fill="1" visible="yes" active="yes"/>
-<layer number="49" name="Reference" color="7" fill="1" visible="yes" active="yes"/>
+<layer number="43" name="vRestrict" color="2" fill="10" visible="no" active="yes"/>
+<layer number="44" name="Drills" color="7" fill="1" visible="no" active="yes"/>
+<layer number="45" name="Holes" color="7" fill="1" visible="no" active="yes"/>
+<layer number="46" name="Milling" color="3" fill="1" visible="no" active="yes"/>
+<layer number="47" name="Measures" color="7" fill="1" visible="no" active="yes"/>
+<layer number="48" name="Document" color="7" fill="1" visible="no" active="yes"/>
+<layer number="49" name="Reference" color="7" fill="1" visible="no" active="yes"/>
 <layer number="51" name="tDocu" color="7" fill="1" visible="yes" active="yes"/>
 <layer number="52" name="bDocu" color="7" fill="1" visible="yes" active="yes"/>
@@
 <param name="mlMinCreamFrame" value="0mil"/>
 <param name="mlMaxCreamFrame" value="0mil"/>
-<param name="mlViaStopLimit" value="0mil"/>
+<param name="mlViaStopLimit" value="11mil"/>
 <param name="srRoundness" value="0"/>
 <param name="srMinRoundness" value="0mil"/>
@@
 <wire x1="19.528" y1="19.274" x2="18.796" y2="18.542" width="0.2032" layer="1"/>
 <via x="18.796" y="18.542" extent="1-16" drill="0.35"/>
-<wire x1="13.344" y1="4.454" x2="13.462" y2="4.572" width="0.2032" layer="16"/>
-<wire x1="8.3247875" y1="4.454" x2="13.344" y2="4.454" width="0.2032" layer="16"/>
-<wire x1="8.3247875" y1="4.454" x2="8.176" y2="4.3052125" width="0.2032" layer="16"/>
-<wire x1="8.176" y1="4.3052125" x2="8.176" y2="3.556" width="0.2032" layer="16"/>
-<wire x1="8.176" y1="3.556" x2="8.176" y2="1.0947875" width="0.2032" layer="16"/>
-<wire x1="8.176" y1="1.0947875" x2="8.3247875" y2="0.946" width="0.2032" layer="16"/>
-<wire x1="8.3247875" y1="0.946" x2="8.4266" y2="0.946" width="0.2032" layer="16"/>
-<wire x1="8.4266" y1="0.946" x2="8.89" y2="0.4826" width="0.2032" layer="16"/>
-<wire x1="18.796" y1="4.572" x2="13.462" y2="4.572" width="0.2032" layer="16"/>
 <wire x1="18.796" y1="4.572" x2="18.796" y2="8.382" width="0.2032" layer="16"/>
 <wire x1="18.796" y1="8.382" x2="18.766" y2="8.412" width="0.2032" layer="16"/>
 <wire x1="18.766" y1="8.412" x2="17.272" y2="8.412" width="0.2032" layer="16"/>
 <wire x1="24.8666" y1="11.4046" x2="24.8666" y2="17.2974" width="0.3048" layer="16"/>
+<wire x1="8.128" y1="4.572" x2="7.874" y2="4.318" width="0.2032" layer="16"/>
+<wire x1="7.874" y1="4.318" x2="7.874" y2="1.016" width="0.2032" layer="16"/>
+<wire x1="7.874" y1="1.016" x2="8.4074" y2="0.4826" width="0.2032" layer="16"/>
+<wire x1="8.4074" y1="0.4826" x2="8.89" y2="0.4826" width="0.2032" layer="16"/>
+<wire x1="18.796" y1="4.572" x2="8.128" y2="4.572" width="0.2032" layer="16"/>
 <wire x1="8.89" y1="0.4826" x2="8.89" y2="0" width="0" layer="19" extent="16-16"/>
 </signal>
